Commit message: Fixed rviz error

File: urdf/agv_v1.xacro (robot description, xacro)
@@ -1,4 +1,4 @@
 <?xml version="1.0"?>
-<robot name="Diff_Drive" xmlns:xacro="http://www.ros.org/wiki/xacro">
+<robot name="agv_v1" xmlns:xacro="http://www.ros.org/wiki/xacro">
 <!-- /////////////////////////////////////////////////////-->
 <material name="Black">
@@ -61,5 +61,5 @@
         <box size="${chassis_length} ${chassis_width} ${chassis_height}"/>
         <!-- mesh filename="$(find agvsim)/meshes/Wheel.igs)"/ -->
-       </geometry>
+      </geometry>
      </visual>
     <collision>
@@ -69,9 +69,6 @@
       </geometry>
     </collision>
-    <xacro:chassis_inertia mass="1.0"/>
+    <xacro:chassis_inertia mass="2.0"/>
  </link>
- <!-- <gazebo reference="base_link">
-    <turnGravityOff>false</turnGravityOff>
- </gazebo> -->
 <!-- ******************* WHEELS ********************* -->
 <xacro:macro name="wheel" params= "prefix suffix X Y Z">
@@ -80,8 +77,8 @@
      <origin rpy= "${PI/2} 0 0" xyz= "0 0 0"/>
      <geometry>
-     	<cylinder length="${wheel_width}" radius= "${wheel_radius}"/>
-     	<!-- mesh filename="$(find agvsim)/meshes/Chassis.igs)"/ -->
+     	<!-- <cylinder length="${wheel_width}" radius= "${wheel_radius}"/> -->
+      <box size="${wheel_radius*2} ${wheel_width} 0.01" />
+      <!-- <mesh filename="$(find agvsim)/meshes/wheel.stl)"/> -->
      </geometry>
-     <mesh filename="$(find agvsim)/meshes/wheel.stl)"/>
      <material name= "Black"/>
     </visual>
@@ -89,26 +86,14 @@
      <origin rpy= "${PI/2} 0 0" xyz= "0 0 0"/>
      <geometry><cylinder length="${wheel_width}" radius= "${wheel_radius}"/></geometry>
-     <surface>
-        <friction>
-          <ode>
-            <mu>100</mu>
-            <mu2>50</mu2>
-            <slip1>1.0</slip1>
-            <slip2>1.0</slip2>
-          </ode>
-        </friction>
-      </surface>
     </collision>
   <xacro:wheel_inertia m="${wheel_mass}" r="${wheel_radius}" h="${wheel_width}"/>
   </link>
-  <!-- <gazebo reference ="${prefix}_${suffix}_wheel">
-     <turnGravityOff>false</turnGravityOff>
-  </gazebo> -->
-  <!-- gazebo reference ="${prefix}_${suffix}_wheel">
-    <mu1 value="${mu1}"/>
-    <mu2 value="${mu2}"/>
-    <kp value="10000000.0"/>
-    <kd value= "1.0"/>
-  </gazebo -->
+  <gazebo reference="{prefix}_${suffix}_wheel">
+    <mu1 value="10000"/>
+    <mu2 value="200000"/>
+    <kp  value="10E2" />
+    <kd  value="1" />
+    <fdir1 value="1 0 0"/>
+  </gazebo>
   <joint name="${prefix}_${suffix}_wheel_joint" type="continuous">
 	  <parent link= "base_link"/>
@@ -116,5 +101,5 @@
 	  <origin xyz= "${chassis_length/2 - wheel_radius} ${(chassis_width/2+wheel_width/2)*Z}  ${wheel_radius}" rpy="0 0 0"/>
 	  <axis xyz="0 1 0"/>
-  	  <limit effort= "10000" velocity="1000"/>
+  	  <!-- <limit effort= "10000" velocity="1000"/> -->
   	  <dynamics damping="1.0" friction="1.0"/>
   </joint>
